File: hardware/bbu-controller/bbu_controller_prototype_kicad/bbu_controller_prototype_kicad.kicad_sch (KiCad schematic)
At the start: 33 parts, among them J1 TERMINAL_BLK, J2 Conn_01x09_Pin, J3 Conn_01x02, J4 Conn_01x02, J5 Conn_01x09_Pin, J6 Conn_01x02, J7 TERMINAL_BLK, M1 Snubber_module_220VAC, M2 JQC-3FE-S-Z_MODULE, M3 TFT 1.8", M4 ZMCT103C, M5 ROTARY_ENC_W/SW_MODULE, M6 ADS1115, M7 ESP32-C3-ZERO, M8 4-24V to 5V buck

Commit message: Record v0.08 protoboard, exports, and bring-up firmware.
Living docs match the soldered board. KiCad v0.08 plus BOM/netlist/ERC
replace the v0.06 exports. node-bbu now drives the relay via Q1, samples
A0–A3, and blinks GPIO8. Issue 009 tracks the offline control loop.
Parts:
- removed TP1: 12V, symbol Connector:TestPoint
- added D1, D2: LED, symbol Device:LED
- added J7: Conn_01x02_Pin, symbol Connector:Conn_01x02_Pin
- added Q1: 2N3904, Package_TO_SOT_THT:TO-92_Inline, symbol Transistor_BJT:2N3904
- added R1: 2K, symbol Device:R
- added R7: 2.2K, Resistor_THT:R_Axial_DIN0207_L6.3mm_D2.5mm_P10.16mm_Horizontal, symbol Device:R
- added R8: 4.7K, Resistor_THT:R_Axial_DIN0207_L6.3mm_D2.5mm_P10.16mm_Horizontal, symbol Device:R
- TP1: renamed from TP2; value 5V -> 5V_VO
- renumbered C6 to C5, C8 to C6, D1 to D3, J7 to J8, R1 to R2, R2 to R3, R3 to R4, R4 to R5, R5 to R6
Connections:
- net +3.3V: now also J2.2 (Pin_2), J5.2 (Pin_2); no longer J2.1 (Pin_1), J5.1 (Pin_1)
- net +5V: now also J7.1 (Pin_1); no longer C6.1, M8.1 (VO+), TP1.1
- net ENC_A: now also J2.3 (Pin_3), J5.3 (Pin_3); no longer J2.7 (Pin_7), J5.7 (Pin_7)
- net ENC_B: now also J2.4 (Pin_4), J5.4 (Pin_4); no longer J2.8 (Pin_8), J5.8 (Pin_8)
- net ENC_SW: now also J2.8 (Pin_8), J5.8 (Pin_8); no longer J2.9 (Pin_9), J5.9 (Pin_9)
- net GND: now also J2.1 (Pin_1), J5.1 (Pin_1), D2.1 (K), Q1.1 (E), R7.1; no longer J2.2 (Pin_2), J5.2 (Pin_2)
- net RELAY: now also R1.2; no longer M2.6 (IN)
- net TFT_AO: now also J2.6 (Pin_6), J5.6 (Pin_6); no longer J2.4 (Pin_4), J5.4 (Pin_4)
- net TFT_RESET: now also J2.5 (Pin_5), J5.5 (Pin_5); no longer J2.3 (Pin_3), J5.3 (Pin_3)
- net TFT_SCK: now also J2.9 (Pin_9), J5.9 (Pin_9); no longer J2.6 (Pin_6), J5.6 (Pin_6)
- net TFT_SDA: now also J2.7 (Pin_7), J5.7 (Pin_7); no longer J2.5 (Pin_5), J5.5 (Pin_5)
- net at C5.1, D3.1 (K), M8.3 (IN+): now also R8.1
- net at M7.12 (GPIO_8): now also D1.2 (A)
- new net: D2.2 (A), R8.2
- new net: Q1.2 (B), R1.1
- new net: M2.6 (IN), Q1.3 (C)
- new net: D1.1 (K), R7.2
- new net +5V_VO: C6.1, J7.2 (Pin_2), M8.1 (VO+), TP1.1
- no-connect marks 9 -> 8
Other:
- note added: "USB safety jumper"
- moved on the sheet: C5, C6, D3, F1, J8, M8, TP1
