File: hardware/bbu-controller/bbu_controller_prototype_kicad/bbu_controller_prototype.kicad_sch (KiCad schematic)
At the start: 41 parts, among them J1 TERMINAL_BLK, J2 Conn_01x09_Pin, J3 Conn_01x02, J4 Conn_01x02, J5 Conn_01x09_Pin, J6 Conn_01x02, J7 Conn_01x02_Pin, J8 TERMINAL_BLK, J9 Conn_01x02_Socket, M1 Snubber_module_220VAC, M5 ROTARY_ENC_W/SW_MODULE, Q1 2N3904

Commit message: hardware: schematic v0.09 — encoder A/B/SW caps (bench ISR-storm fix), PPTC F1 omitted (deploy decision 012), CT+snubber already dropped (014); v0.09 exports replace v0.08
Parts:
- removed C7, C8: 100 nF, symbol Device:C_Small_US
- removed M1: Snubber_module_220VAC, symbol 01_my_custom_library:SNUBBER_MODULE
- removed M2: (no value), symbol 01_my_custom_library:RELAY_MODULE
- removed M3: (no value), symbol 01_my_custom_library:1.8{dblquote}_TFT_MODULE
- removed M4: (no value), symbol 01_my_custom_library:ZMCT_COIL_MODULE
- removed M5: ROTARY_ENC_W/SW_MODULE, symbol 01_my_custom_library:ROTARY_ENC_W/SW_MODULE
- removed M6: (no value), symbol 01_my_custom_library:ADC_4CH_MODULE
- removed M7: (no value), symbol 01_my_custom_library:ESP32-C3_ZERO_MODULE
- removed M8: (no value), symbol 01_my_custom_library:BUCK_6-24V_to_5V_MODULE
- added M1: Snubber_module_220VAC, symbol 0_my_custom_library:SNUBBER_MODULE
- added M2: JQC-3FE-S-Z_MODULE, symbol 0_my_custom_library:RELAY_MODULE
- added M3: TFT 1.8", symbol 0_my_custom_library:1.8{dblquote}_TFT_MODULE
- added M4: ZMCT103C, symbol 0_my_custom_library:ZMCT_COIL_MODULE
- added M5: ROTARY_ENC_W/SW_MODULE, symbol 0_my_custom_library:ROTARY_ENC_W/SW_MODULE
- added M6: ADS1115, symbol 0_my_custom_library:ADC_4CH_MODULE
- added M7: ESP32-C3-ZERO, symbol 0_my_custom_library:ESP32-C3_ZERO_MODULE
- added M8: 4-24V to 5V buck, symbol 0_my_custom_library:BUCK_6-24V_to_5V_MODULE
Connections:
- net +3.3V: now also M3.1 (VCC), M3.8 (LED), M4.1 (VCC), M5.4 (VCC), M6.1 (VDD), M7.3 (3v3)
- net +5V: now also M2.4 (VCC), M7.1 (5V)
- net +5V_VO: now also M8.1 (VO+)
- net ADC_SCL: now also M6.3 (SCL), M7.10 (GPIO_6)
- net ADC_SDA: now also M6.4 (SDA), M7.11 (GPIO_7)
- net ENC_A: now also M5.1 (A), M7.4 (GPIO_0)
- net ENC_B: now also M5.3 (B), M7.5 (GPIO_1)
- net ENC_SW: now also M5.6 (SW), M7.9 (GPIO_5)
- net GND: now also M2.5 (GND), M3.2 (GND), M3.3 (CS), M4.3 (GND), M4.4 (GND), M5.5 (GND), M6.2 (GND), M7.2 (GND), M8.2 (GND)
- net RELAY: now also M7.14 (GPIO_10)
- net TFT_AO: now also M3.5 (AO), M7.7 (GPIO_3)
- net TFT_RESET: now also M3.4 (RESET), M7.6 (GPIO_2)
- net TFT_SCK: now also M3.7 (SCK), M7.13 (GPIO_9)
- net TFT_SDA: now also M3.6 (SDA), M7.8 (GPIO_4)
- net at J3.2 (Pin_2), R4.1, TH1.2: now also M6.8 (A1)
- net at J1.1 (Pin_1): now also M1.1 (snub1), M2.1 (NO)
- net at J1.2 (Pin_2): now also M1.2 (snub2), M2.2 (COM)
- net at J6.2 (Pin_2), R6.1, TH3.2: now also M6.10 (A3)
- net at J4.2 (Pin_2), R5.1, TH2.2: now also M6.9 (A2)
- net at C5.1, D3.1 (K), R8.1: now also M8.3 (IN+)
- net at D1.2 (A): now also M7.12 (GPIO_8)
- net at Q1.3 (C): now also M2.6 (IN)
- net at J8.1 (Pin_1): now also F1.1; no longer D3.2 (A)
- net at F1.2: now also D3.2 (A)
- new net: M4.2 (OUT), M6.7 (A0)
- no-connect marks 14 -> 8
Other:
- moved on the sheet: F1, J2, J7
